File: Schematic/V1/V1.kicad_sch (KiCad schematic)
At the start: 15 parts, among them U1 L293D_Motor_Shield

Commit message: Updated schem
Connections:
- net Matrix_CLK: now also XA1.D51; no longer XA1.A13
- net Matrix_CS: now also XA1.D53 (D53_SS); no longer XA1.A14
- net Matrix_DIN: now also XA1.D50; no longer XA1.A15
- new net A14: XA1.A14
- new net A15: XA1.A15
Other:
- moved on the sheet: LB1, LF1, RB1, RF1, Ultrasonic_Front1, Ultrasonic_Front2, Ultrasonic_Front3
